File: HW/mpu_rom_ram.sch (KiCad schematic (older format))
At the start: 11 parts, among them U1 WD65C816S_PLCC44, U2 AS7C34096A, U5 AS6C62256A, U6 AS7C34096A

Commit message: Removed two ram chips, down to 1 MiB.
Parts:
- added C23, C24, C25, C26: 0.1uF, Capacitors_ThroughHole:C_Disc_D4.7mm_W2.5mm_P5.00mm, symbol device:C_Small
- added U13, U14: AS7C34096A, saturn:SOJ-36, symbol pluto:AS7C34096A
- C10, C11, C12, C13, C7, C8, C9: symbol C_Small -> device:C_Small
- U1: symbol WD65C816S_PLCC44 -> 65xx:WD65C816S_PLCC44
- U2, U6: footprint Housings_SOIC:SOIC-28W_7.5x18.7mm_Pitch1.27mm -> saturn:SOJ-36; symbol AS7C34096A -> pluto:AS7C34096A
- U5: symbol AS6C62256A -> pluto:AS6C62256A
Connections:
- net A0: now also U13.1 (A0), U14.1 (A0)
- net A1: now also U13.2 (A1), U14.2 (A1)
- net A10: now also U13.20 (A10), U14.20 (A10)
- net A11: now also U13.21 (A11), U14.21 (A11)
- net A12: now also U13.22 (A12), U14.22 (A12)
- net A13: now also U13.23 (A13), U14.23 (A13)
- net A14: now also U13.24 (A14), U14.24 (A14)
- net A15: now also U13.32 (A15), U14.32 (A15)
- net A16: now also U13.33 (A16), U14.33 (A16)
- net A17: now also U13.34 (A17), U14.34 (A17)
- net A18: now also U13.35 (A18), U14.35 (A18)
- net A2: now also U13.3 (A2), U14.3 (A2)
- net A3: now also U13.4 (A3), U14.4 (A3)
- net A4: now also U13.5 (A4), U14.5 (A4)
- net A5: now also U13.14 (A5), U14.14 (A5)
- net A6: now also U13.15 (A6), U14.15 (A6)
- net A7: now also U13.16 (A7), U14.16 (A7)
- net A8: now also U13.17 (A8), U14.17 (A8)
- net A9: now also U13.18 (A9), U14.18 (A9)
- net D0: now also U13.7 (I/O1), U14.7 (I/O1)
- net D1: now also U13.8 (I/O2), U14.8 (I/O2)
- net D2: now also U13.11 (I/O3), U14.11 (I/O3)
- net D3: now also U13.12 (I/O4), U14.12 (I/O4)
- net D4: now also U13.25 (I/O5), U14.25 (I/O5)
- net D5: now also U13.26 (I/O6), U14.26 (I/O6)
- net D6: now also U13.29 (I/O7), U14.29 (I/O7)
- net D7: now also U13.30 (I/O8), U14.30 (I/O8)
- net GND: now also C23.1, C24.2, C25.1, C26.2, U13.10 (GND), U13.28 (GND), U14.10 (GND), U14.28 (GND)
- net VCC: now also C23.2, C24.1, C25.2, C26.1, U13.27 (VCC), U13.9 (VCC), U14.27 (VCC), U14.9 (VCC)
- net ~MRD: now also U13.31 (~OE), U14.31 (~OE)
- net ~MWR: now also U13.13 (~WE), U14.13 (~WE)
- new net ~RAM2: U14.6 (~CE)
- new net ~RAM3: U13.6 (~CE)
Other:
- note added: "RAM0 (00:0000-07:FFFF)"
- note added: "RAM1 (08:0000-0F:FFFF)"
- note added: "RAM2 (10:0000-17:FFFF)"
- note added: "RAM3 (18:0000-1F:FFFF)"
- note added: "ROM (00:8000-00:FFFF)"
- note removed: "RAM (000000-07FFFF)"
- note removed: "RAM (080000-0FFFFF)"
