File: HW/mpu_rom_ram.sch (KiCad schematic (older format))
At the start: 11 parts, among them U1 WD65C816S_PLCC44, U2 AS7C34096A, U5 AS6C62256A, U6 AS7C34096A

Commit message: Fixed bus error in RTC design.
Parts:
- C10, C11, C12, C13, C7, C8, C9: symbol device:C_Small -> saturn-rescue:C_Small-device
- U1: symbol 65xx:WD65C816S_PLCC44 -> saturn-rescue:WD65C816S_PLCC44-65xx
Changed lines of the file:
@@
 EESchema Schematic File Version 4
 LIBS:saturn-cache
-EELAYER 26 0
+EELAYER 29 0
 EELAYER END
 $Descr A4 11693 8268
@@
 	5125 2925 4800 2925
 $Comp
-L 65xx:WD65C816S_PLCC44 U1
+L saturn-rescue:WD65C816S_PLCC44-65xx U1
 U 1 1 5A3AB10B
 P 2600 2375
+AR Path="/5A3AB10B" Ref="U1"  Part="1"
+AR Path="/5952FC78/5A3AB10B" Ref="U1"  Part="1"
 F 0 "U1" H 2975 3400 60  0000 C CNN
 F 1 "WD65C816S_PLCC44" V 2600 2275 60  0000 C CNN
@@
 $EndComp
 $Comp
-L device:C_Small C12
+L saturn-rescue:C_Small-device C12
 U 1 1 5A3AB89B
 P 8725 3600
@@
 $EndComp
 $Comp
-L device:C_Small C10
+L saturn-rescue:C_Small-device C10
 U 1 1 5A3AB916
 P 7350 3600
@@
 $EndComp
 $Comp
-L device:C_Small C9
+L saturn-rescue:C_Small-device C9
 U 1 1 5A3AB953
 P 6025 3275
@@
 $EndComp
 $Comp
-L device:C_Small C8
+L saturn-rescue:C_Small-device C8
 U 1 1 5A3ABA08
 P 3275 1125
@@
 $EndComp
 $Comp
-L device:C_Small C7
+L saturn-rescue:C_Small-device C7
 U 1 1 5A3ABA2D
 P 2000 1125
@@
 $EndComp
 $Comp
-L power1:GND #PWR01
+L saturn-rescue:GND-power1 #PWR01
 U 1 1 5A3AC09F
 P 2600 3900
@@
 	7425 6100 7100 6100
 $Comp
-L device:C_Small C13
+L saturn-rescue:C_Small-device C13
 U 1 1 5A3C0579
 P 8750 6375
@@
 $EndComp
 $Comp
-L device:C_Small C11
+L saturn-rescue:C_Small-device C11
 U 1 1 5A3C057F
 P 7350 6375
@@
 	6050 2725 6350 2725
 $Comp
-L power1:VCC #PWR02
+L saturn-rescue:VCC-power1 #PWR02
 U 1 1 5A3F84C5
 P 6350 2725
@@
 RAM1 (08:0000-0F:FFFF)
 $Comp
-L power1:GND #PWR03
+L saturn-rescue:GND-power1 #PWR03
 U 1 1 5AA65D61
 P 2700 3900
@@
 $EndComp
 $Comp
-L power1:GND #PWR04
+L saturn-rescue:GND-power1 #PWR04
 U 1 1 5AA65D8B
 P 2500 3900
@@
 Connection ~ 2700 3850
 $Comp
-L power1:VCC #PWR05
+L saturn-rescue:VCC-power1 #PWR05
 U 1 1 5AA1A97C
 P 7925 1225
@@
 $EndComp
 $Comp
-L power1:VCC #PWR06
+L saturn-rescue:VCC-power1 #PWR06
 U 1 1 5AA1AA07
 P 8125 1225
@@
 $EndComp
 $Comp
-L power1:VCC #PWR07
+L saturn-rescue:VCC-power1 #PWR07
 U 1 1 5AA1AA9D
 P 7925 4000
@@
 $EndComp
 $Comp
-L power1:VCC #PWR08
+L saturn-rescue:VCC-power1 #PWR08
 U 1 1 5AA1AAC5
 P 8125 4000
@@
 $EndComp
 $Comp
-L power1:VCC #PWR09
+L saturn-rescue:VCC-power1 #PWR09
 U 1 1 5AA1AB85
 P 2500 1125
@@
 $EndComp
 $Comp
-L power1:VCC #PWR010
+L saturn-rescue:VCC-power1 #PWR010
 U 1 1 5AA1ABAB
 P 2700 1125
@@
 $EndComp
 $Comp
-L power1:GND #PWR011
+L saturn-rescue:GND-power1 #PWR011
 U 1 1 5AA1AC83
 P 7925 3600
@@
 $EndComp
 $Comp
-L power1:GND #PWR012
+L saturn-rescue:GND-power1 #PWR012
 U 1 1 5AA1ACAB
 P 8125 3600
@@
 $EndComp
 $Comp
-L power1:GND #PWR013
+L saturn-rescue:GND-power1 #PWR013
 U 1 1 5AA1AD6D
 P 7925 6375
@@
 $EndComp
 $Comp
-L power1:GND #PWR014
+L saturn-rescue:GND-power1 #PWR014
 U 1 1 5AA1AD95
 P 8125 6375
@@
 $EndComp
 $Comp
-L power1:GND #PWR015
+L saturn-rescue:GND-power1 #PWR015
 U 1 1 5AA1AED9
 P 5600 3275
@@
 $EndComp
 $Comp
-L power1:VCC #PWR016
+L saturn-rescue:VCC-power1 #PWR016
 U 1 1 5AA1AF59
 P 5600 1275

Commit message: Cosmetic changes to schema. Parking this project as router can't find a route.
Parts:
- U1: footprint saturn:PLCC-44_THT-Socket -> Package_LCC:PLCC-44_THT-Socket
- U2, U6: footprint saturn:SOJ-36 -> Grotto:SOJ-36
Changed lines of the file:
@@
 F 0 "U2" H 8275 3500 60  0000 C CNN
 F 1 "AS7C34096A" V 8025 2025 60  0000 C CNN
-F 2 "saturn:SOJ-36" H 8025 2425 60  0001 C CNN
+F 2 "Grotto:SOJ-36" H 8025 2425 60  0001 C CNN
 F 3 "" H 8025 2425 60  0001 C CNN
 	1    8025 2425
@@
 F 0 "U1" H 2975 3400 60  0000 C CNN
 F 1 "WD65C816S_PLCC44" V 2600 2275 60  0000 C CNN
-F 2 "saturn:PLCC-44_THT-Socket" H 1975 1475 60  0001 C CNN
+F 2 "Package_LCC:PLCC-44_THT-Socket" H 1975 1475 60  0001 C CNN
 F 3 "" H 1975 1475 60  0000 C CNN
 	1    2600 2375
@@
 F 0 "U6" H 8275 6275 60  0000 C CNN
 F 1 "AS7C34096A" V 8025 4800 60  0000 C CNN
-F 2 "saturn:SOJ-36" H 8025 5200 60  0001 C CNN
+F 2 "Grotto:SOJ-36" H 8025 5200 60  0001 C CNN
 F 3 "" H 8025 5200 60  0001 C CNN
 	1    8025 5200
