File: HW/via_and_ide.sch (KiCad schematic (older format))
At the start: 6 parts, among them J3 VIA2PB, J4 IDE, U7 WD65C22PLCC44, U8 WD65C22PLCC44

Commit message: Added address decoding.
Connections:
- net GND: now also J3.1 (P1), J3.2 (P2); no longer J3.13 (P13), J3.14 (P14)
- net VCC: now also J3.13 (P13), J3.14 (P14); no longer J3.1 (P1), J3.2 (P2)
Changed lines of the file:
@@
 L VCC #PWR?
 U 1 1 5A3E3F24
-P 6200 2875
-F 0 "#PWR?" H 6200 2725 50  0001 C CNN
-F 1 "VCC" H 6200 3025 50  0000 C CNN
-F 2 "" H 6200 2875 50  0001 C CNN
-F 3 "" H 6200 2875 50  0001 C CNN
-	1    6200 2875
-	1    0    0    -1
+P 6200 3925
+F 0 "#PWR?" H 6200 3775 50  0001 C CNN
+F 1 "VCC" H 6200 4075 50  0000 C CNN
+F 2 "" H 6200 3925 50  0001 C CNN
+F 3 "" H 6200 3925 50  0001 C CNN
+	1    6200 3925
+	-1   0    0    1
 $EndComp
 $Comp
 L GND #PWR?
 U 1 1 5A3E3F44
-P 6200 3925
-F 0 "#PWR?" H 6200 3675 50  0001 C CNN
-F 1 "GND" H 6200 3775 50  0000 C CNN
-F 2 "" H 6200 3925 50  0001 C CNN
-F 3 "" H 6200 3925 50  0001 C CNN
-	1    6200 3925
-	1    0    0    -1
+P 6200 2875
+F 0 "#PWR?" H 6200 2625 50  0001 C CNN
+F 1 "GND" H 6200 2725 50  0000 C CNN
+F 2 "" H 6200 2875 50  0001 C CNN
+F 3 "" H 6200 2875 50  0001 C CNN
+	1    6200 2875
+	-1   0    0    1
 $EndComp
 NoConn ~ 2225 2350

Commit message: Simulation of address decoding.
Parts:
- added D2, D3: D, symbol D
- gave numbers to parts that had none: 2
Connections:
- net ~IRQ: now also D2.2 (A), D3.2 (A); no longer U7.23 (~IRQ), U8.23 (~IRQ)
- new net: D2.1 (K), U7.23 (~IRQ)
- new net: D3.1 (K), U8.23 (~IRQ)
Changed lines of the file:
@@
 	8950 2425 9050 2525
 Text HLabel 9050 4900 2    60   Input ~ 0
-A[0..18]
+A[0..19]
 Text Label 8950 2425 2    60   ~ 0
 A0
@@
 A3
 Text Label 7675 4900 2    60   ~ 0
-A[0..18]
+A[0..19]
 Text Label 3950 2425 2    60   ~ 0
 A0
@@
 Text HLabel 8775 3800 2    60   Input ~ 0
 ~RES
-Text HLabel 8775 3925 2    60   Output ~ 0
+Text HLabel 9275 3925 2    60   Output ~ 0
 ~IRQ
 Text HLabel 8775 3550 2    60   Input ~ 0
@@
 Text HLabel 3775 3800 2    60   Input ~ 0
 ~RES
-Text HLabel 3775 3925 2    60   Output ~ 0
+Text HLabel 4275 3925 2    60   Output ~ 0
 ~IRQ
 Text HLabel 3775 3550 2    60   Input ~ 0
@@
 ~VIA2SEL
 $Comp
-L VCC #PWR?
+L VCC #PWR16
 U 1 1 5A3DECA8
 P 3950 3000
-F 0 "#PWR?" H 3950 2850 50  0001 C CNN
+F 0 "#PWR16" H 3950 2850 50  0001 C CNN
 F 1 "VCC" H 3850 3075 50  0000 C CNN
 F 2 "" H 3950 3000 50  0001 C CNN
@@
 $EndComp
 $Comp
-L VCC #PWR?
+L VCC #PWR23
 U 1 1 5A3DEEFA
 P 8950 3000
-F 0 "#PWR?" H 8950 2850 50  0001 C CNN
+F 0 "#PWR23" H 8950 2850 50  0001 C CNN
 F 1 "VCC" H 8850 3075 50  0000 C CNN
 F 2 "" H 8950 3000 50  0001 C CNN
@@
 $EndComp
 $Comp
-L GND #PWR?
+L GND #PWR22
 U 1 1 5A3DF2AF
 P 7950 4625
-F 0 "#PWR?" H 7950 4375 50  0001 C CNN
+F 0 "#PWR22" H 7950 4375 50  0001 C CNN
 F 1 "GND" H 7950 4475 50  0000 C CNN
 F 2 "" H 7950 4625 50  0001 C CNN
@@
 $EndComp
 $Comp
-L GND #PWR?
+L GND #PWR14
 U 1 1 5A3DF646
 P 2950 4625
-F 0 "#PWR?" H 2950 4375 50  0001 C CNN
+F 0 "#PWR14" H 2950 4375 50  0001 C CNN
 F 1 "GND" H 2950 4475 50  0000 C CNN
 F 2 "" H 2950 4625 50  0001 C CNN
@@
 $EndComp
 $Comp
-L VCC #PWR?
+L VCC #PWR21
 U 1 1 5A3DFA06
 P 7950 875
-F 0 "#PWR?" H 7950 725 50  0001 C CNN
+F 0 "#PWR21" H 7950 725 50  0001 C CNN
 F 1 "VCC" H 7850 950 50  0000 C CNN
 F 2 "" H 7950 875 50  0001 C CNN
@@
 $EndComp
 $Comp
-L VCC #PWR?
+L VCC #PWR13
 U 1 1 5A3DFA22
 P 2950 875
-F 0 "#PWR?" H 2950 725 50  0001 C CNN
+F 0 "#PWR13" H 2950 725 50  0001 C CNN
 F 1 "VCC" H 2950 1025 50  0000 C CNN
 F 2 "" H 2950 875 50  0001 C CNN
@@
 $EndComp
 $Comp
-L C_Small C?
+L C_Small C17
 U 1 1 5A3DFACE
 P 8375 925
-F 0 "C?" V 8500 875 50  0000 L CNN
+F 0 "C17" V 8500 875 50  0000 L CNN
 F 1 "0.1uF" V 8250 850 50  0000 L CNN
 F 2 "" H 8375 925 50  0001 C CNN
@@
 $EndComp
 $Comp
-L C_Small C?
+L C_Small C16
 U 1 1 5A3DFDF6
 P 3275 925
-F 0 "C?" V 3375 875 50  0000 L CNN
+F 0 "C16" V 3375 875 50  0000 L CNN
 F 1 "0.1uF" V 3150 825 50  0000 L CNN
 F 2 "" H 3275 925 50  0001 C CNN
@@
 IDE-D15
 $Comp
-L VCC #PWR?
+L VCC #PWR20
 U 1 1 5A3E3F24
 P 6200 3925
-F 0 "#PWR?" H 6200 3775 50  0001 C CNN
+F 0 "#PWR20" H 6200 3775 50  0001 C CNN
 F 1 "VCC" H 6200 4075 50  0000 C CNN
 F 2 "" H 6200 3925 50  0001 C CNN
@@
 $EndComp
 $Comp
-L GND #PWR?
+L GND #PWR19
 U 1 1 5A3E3F44
 P 6200 2875
-F 0 "#PWR?" H 6200 2625 50  0001 C CNN
+F 0 "#PWR19" H 6200 2625 50  0001 C CNN
 F 1 "GND" H 6200 2725 50  0000 C CNN
 F 2 "" H 6200 2875 50  0001 C CNN
@@
 ~IDE:CS1
 $Comp
-L GND #PWR?
+L GND #PWR18
 U 1 1 5A3E84F7
 P 5175 7250
-F 0 "#PWR?" H 5175 7000 50  0001 C CNN
+F 0 "#PWR18" H 5175 7000 50  0001 C CNN
 F 1 "GND" H 5175 7100 50  0000 C CNN
 F 2 "" H 5175 7250 50  0001 C CNN
@@
 IDE-A2
 $Comp
-L GND #PWR?
+L GND #PWR17
 U 1 1 5A3E9E8F
 P 4975 5275
-F 0 "#PWR?" H 4975 5025 50  0001 C CNN
+F 0 "#PWR17" H 4975 5025 50  0001 C CNN
 F 1 "GND" H 4975 5125 50  0000 C CNN
 F 2 "" H 4975 5275 50  0001 C CNN
@@
 NoConn ~ 3875 6275
 $Comp
-L GND #PWR?
+L GND #PWR15
 U 1 1 5A3ECBDD
 P 3275 6175
-F 0 "#PWR?" H 3275 5925 50  0001 C CNN
+F 0 "#PWR15" H 3275 5925 50  0001 C CNN
 F 1 "GND" H 3275 6025 50  0000 C CNN
 F 2 "" H 3275 6175 50  0001 C CNN
@@
 Text Label 2575 5125 0    60   ~ 0
 ~IDE:RES
+$Comp
+L D D2
+U 1 1 5A458E7D
+P 3925 3925
+F 0 "D2" H 3925 3850 50  0000 C CNN
+F 1 "D" H 4000 3900 50  0000 C CNN
+F 2 "" H 3925 3925 50  0001 C CNN
+F 3 "" H 3925 3925 50  0001 C CNN
+	1    3925 3925
+	1    0    0    -1
+$EndComp
+Wire Wire Line
+	4075 3925 4275 3925
+$Comp
+L D D3
+U 1 1 5A4591CE
+P 8925 3925
+F 0 "D3" H 8925 3850 50  0000 C CNN
+F 1 "D" H 9000 3900 50  0000 C CNN
+F 2 "" H 8925 3925 50  0001 C CNN
+F 3 "" H 8925 3925 50  0001 C CNN
+	1    8925 3925
+	1    0    0    -1
+$EndComp
+Wire Wire Line
+	9075 3925 9275 3925
 $EndSCHEMATC

Commit message: ABEL code passes compilation, no tests though. Small changes to schema
Parts:
- added D4: LED, LEDs:LED_D3.0mm, symbol LED
- added R6, R7: 3.3k, Resistors_ThroughHole:R_Axial_DIN0207_L6.3mm_D2.5mm_P2.54mm_Vertical, symbol R_Small
- C16, C17: footprint (none) -> Capacitors_ThroughHole:C_Disc_D4.7mm_W2.5mm_P5.00mm
- D2, D3: footprint (none) -> Diodes_ThroughHole:D_DO-35_SOD27_P7.62mm_Horizontal
- J3: footprint (none) -> Connectors_IDC:IDC-Header_2x07_Pitch2.54mm_Straight
- J4: footprint (none) -> Connectors_IDC:IDC-Header_2x20_Pitch2.54mm_Straight
- U7, U8: footprint (none) -> saturn:PLCC-44_THT-Socket
Connections:
- net VCC: now also R6.1, R7.1
- net ~IDE:DASP: now also D4.1 (K)
- net ~IDE:DMACK: now also R6.2
- new net: D4.2 (A), R7.2
Changed lines of the file:
@@
 $Descr A4 11693 8268
 encoding utf-8
-Sheet 4 6
+Sheet 4 7
 Title ""
-Date "2017-12-23"
+Date "2018-01-17"
 Rev "0.1"
 Comp "Linux Grotto"
@@
 F 0 "U7" H 2675 3375 60  0000 C CNN
 F 1 "WD65C22PLCC44" V 2950 1600 60  0000 C CNN
-F 2 "" H 2375 2325 60  0000 C CNN
+F 2 "saturn:PLCC-44_THT-Socket" H 2375 2325 60  0001 C CNN
 F 3 "" H 2375 2325 60  0000 C CNN
 	1    2875 2300
@@
 F 0 "U8" H 7675 3375 60  0000 C CNN
 F 1 "WD65C22PLCC44" V 7950 1600 60  0000 C CNN
-F 2 "" H 7375 2325 60  0000 C CNN
+F 2 "saturn:PLCC-44_THT-Socket" H 7375 2325 60  0001 C CNN
 F 3 "" H 7375 2325 60  0000 C CNN
 	1    7875 2300
@@
 F 0 "J4" H 4125 7275 50  0000 C CNN
 F 1 "IDE" V 4125 6225 50  0000 C CNN
-F 2 "" H 4125 5275 50  0001 C CNN
+F 2 "Connectors_IDC:IDC-Header_2x20_Pitch2.54mm_Straight" H 4125 5275 50  0001 C CNN
 F 3 "" H 4125 5275 50  0001 C CNN
 	1    4125 6225
@@
 F 0 "J3" H 6200 3850 50  0000 C CNN
 F 1 "VIA2PB" V 6200 3450 50  0000 C CNN
-F 2 "" H 6200 2250 50  0001 C CNN
+F 2 "Connectors_IDC:IDC-Header_2x07_Pitch2.54mm_Straight" H 6200 2250 50  0001 C CNN
 F 3 "" H 6200 2250 50  0001 C CNN
 	1    6200 3450
@@
 	8950 2425 9050 2525
 Text HLabel 9050 4900 2    60   Input ~ 0
-A[0..19]
+A[0..18]
 Text Label 8950 2425 2    60   ~ 0
 A0
@@
 ~VIA2SEL
 $Comp
-L VCC #PWR16
+L VCC #PWR028
 U 1 1 5A3DECA8
 P 3950 3000
-F 0 "#PWR16" H 3950 2850 50  0001 C CNN
+F 0 "#PWR028" H 3950 2850 50  0001 C CNN
 F 1 "VCC" H 3850 3075 50  0000 C CNN
 F 2 "" H 3950 3000 50  0001 C CNN
@@
 $EndComp
 $Comp
-L VCC #PWR23
+L VCC #PWR029
 U 1 1 5A3DEEFA
 P 8950 3000
-F 0 "#PWR23" H 8950 2850 50  0001 C CNN
+F 0 "#PWR029" H 8950 2850 50  0001 C CNN
 F 1 "VCC" H 8850 3075 50  0000 C CNN
 F 2 "" H 8950 3000 50  0001 C CNN
@@
 $EndComp
 $Comp
-L GND #PWR22
+L GND #PWR030
 U 1 1 5A3DF2AF
 P 7950 4625
-F 0 "#PWR22" H 7950 4375 50  0001 C CNN
+F 0 "#PWR030" H 7950 4375 50  0001 C CNN
 F 1 "GND" H 7950 4475 50  0000 C CNN
 F 2 "" H 7950 4625 50  0001 C CNN
@@
 $EndComp
 $Comp
-L GND #PWR14
+L GND #PWR031
 U 1 1 5A3DF646
 P 2950 4625
-F 0 "#PWR14" H 2950 4375 50  0001 C CNN
+F 0 "#PWR031" H 2950 4375 50  0001 C CNN
 F 1 "GND" H 2950 4475 50  0000 C CNN
 F 2 "" H 2950 4625 50  0001 C CNN
@@
 $EndComp
 $Comp
-L VCC #PWR21
+L VCC #PWR032
 U 1 1 5A3DFA06
 P 7950 875
-F 0 "#PWR21" H 7950 725 50  0001 C CNN
+F 0 "#PWR032" H 7950 725 50  0001 C CNN
 F 1 "VCC" H 7850 950 50  0000 C CNN
 F 2 "" H 7950 875 50  0001 C CNN
@@
 $EndComp
 $Comp
-L VCC #PWR13
+L VCC #PWR033
 U 1 1 5A3DFA22
 P 2950 875
-F 0 "#PWR13" H 2950 725 50  0001 C CNN
+F 0 "#PWR033" H 2950 725 50  0001 C CNN
 F 1 "VCC" H 2950 1025 50  0000 C CNN
 F 2 "" H 2950 875 50  0001 C CNN
@@
 F 0 "C17" V 8500 875 50  0000 L CNN
 F 1 "0.1uF" V 8250 850 50  0000 L CNN
-F 2 "" H 8375 925 50  0001 C CNN
+F 2 "Capacitors_ThroughHole:C_Disc_D4.7mm_W2.5mm_P5.00mm" H 8375 925 50  0001 C CNN
 F 3 "" H 8375 925 50  0001 C CNN
 	1    8375 925
@@
 F 0 "C16" V 3375 875 50  0000 L CNN
 F 1 "0.1uF" V 3150 825 50  0000 L CNN
-F 2 "" H 3275 925 50  0001 C CNN
+F 2 "Capacitors_ThroughHole:C_Disc_D4.7mm_W2.5mm_P5.00mm" H 3275 925 50  0001 C CNN
 F 3 "" H 3275 925 50  0001 C CNN
 	1    3275 925
@@
 IDE-D15
 $Comp
-L VCC #PWR20
+L VCC #PWR034
 U 1 1 5A3E3F24
 P 6200 3925
-F 0 "#PWR20" H 6200 3775 50  0001 C CNN
+F 0 "#PWR034" H 6200 3775 50  0001 C CNN
 F 1 "VCC" H 6200 4075 50  0000 C CNN
 F 2 "" H 6200 3925 50  0001 C CNN
@@
 $EndComp
 $Comp
-L GND #PWR19
+L GND #PWR035
 U 1 1 5A3E3F44
 P 6200 2875
-F 0 "#PWR19" H 6200 2625 50  0001 C CNN
+F 0 "#PWR035" H 6200 2625 50  0001 C CNN
 F 1 "GND" H 6200 2725 50  0000 C CNN
 F 2 "" H 6200 2875 50  0001 C CNN
@@
 ~IDE:CS1
 $Comp
-L GND #PWR18
+L GND #PWR036
 U 1 1 5A3E84F7
 P 5175 7250
-F 0 "#PWR18" H 5175 7000 50  0001 C CNN
+F 0 "#PWR036" H 5175 7000 50  0001 C CNN
 F 1 "GND" H 5175 7100 50  0000 C CNN
 F 2 "" H 5175 7250 50  0001 C CNN
@@
 IDE-A2
 $Comp
-L GND #PWR17
+L GND #PWR037
 U 1 1 5A3E9E8F
 P 4975 5275
-F 0 "#PWR17" H 4975 5025 50  0001 C CNN
+F 0 "#PWR037" H 4975 5025 50  0001 C CNN
 F 1 "GND" H 4975 5125 50  0000 C CNN
 F 2 "" H 4975 5275 50  0001 C CNN
@@
 	3875 6475 3275 6475
 Wire Wire Line
-	3875 6675 3275 6675
+	2275 6675 3875 6675
 Wire Wire Line
 	3875 6775 3275 6775
@@
 	3875 7075 3275 7075
 Wire Wire Line
-	3875 7175 3275 7175
+	3125 7175 3875 7175
 Wire Wire Line
 	4375 5275 4975 5275
@@
 	6825 1500 6925 1600
 Wire Bus Line
-	6825 1500 6825 1250
+	6825 1250 6825 1500
 Wire Bus Line
 	6825 1250 6225 1250
@@
 NoConn ~ 3875 6275
 $Comp
-L GND #PWR15
+L GND #PWR038
 U 1 1 5A3ECBDD
 P 3275 6175
-F 0 "#PWR15" H 3275 5925 50  0001 C CNN
+F 0 "#PWR038" H 3275 5925 50  0001 C CNN
 F 1 "GND" H 3275 6025 50  0000 C CNN
 F 2 "" H 3275 6175 50  0001 C CNN
@@
 F 0 "D2" H 3925 3850 50  0000 C CNN
 F 1 "D" H 4000 3900 50  0000 C CNN
-F 2 "" H 3925 3925 50  0001 C CNN
+F 2 "Diodes_ThroughHole:D_DO-35_SOD27_P7.62mm_Horizontal" H 3925 3925 50  0001 C CNN
 F 3 "" H 3925 3925 50  0001 C CNN
 	1    3925 3925
@@
 F 0 "D3" H 8925 3850 50  0000 C CNN
 F 1 "D" H 9000 3900 50  0000 C CNN
-F 2 "" H 8925 3925 50  0001 C CNN
+F 2 "Diodes_ThroughHole:D_DO-35_SOD27_P7.62mm_Horizontal" H 8925 3925 50  0001 C CNN
 F 3 "" H 8925 3925 50  0001 C CNN
 	1    8925 3925
@@
 Wire Wire Line
 	9075 3925 9275 3925
+$Comp
+L LED D4
+U 1 1 5AA70441
+P 2500 6925
+F 0 "D4" H 2500 7025 50  0000 C CNN
+F 1 "LED" H 2500 6825 50  0000 C CNN
+F 2 "LEDs:LED_D3.0mm" H 2500 6925 50  0001 C CNN
+F 3 "" H 2500 6925 50  0001 C CNN
+	1    2500 6925
+	-1   0    0    1
+$EndComp
+Wire Wire Line
+	2650 6925 3125 6925
+Wire Wire Line
+	2275 6925 2350 6925
+Text Label 3125 6675 2    60   ~ 0
+~IDE:DMACK
+Text Label 3125 6925 2    60   ~ 0
+~IDE:DASP
+Wire Wire Line
+	1950 6475 1950 6925
+$Comp
+L VCC #PWR039
+U 1 1 5AA712EE
+P 1950 6475
+F 0 "#PWR039" H 1950 6325 50  0001 C CNN
+F 1 "VCC" H 1950 6625 50  0000 C CNN
+F 2 "" H 1950 6475 50  0001 C CNN
+F 3 "" H 1950 6475 50  0001 C CNN
+	1    1950 6475
+	1    0    0    -1
+$EndComp
+$Comp
+L R_Small R6
+U 1 1 5AA72016
+P 2175 6675
+F 0 "R6" V 2250 6625 50  0000 L CNN
+F 1 "3.3k" V 2100 6575 50  0000 L CNN
+F 2 "Resistors_ThroughHole:R_Axial_DIN0207_L6.3mm_D2.5mm_P2.54mm_Vertical" H 2175 6675 50  0001 C CNN
+F 3 "" H 2175 6675 50  0001 C CNN
+	1    2175 6675
+	0    -1   -1   0
+$EndComp
+$Comp
+L R_Small R7
+U 1 1 5AA72069
+P 2175 6925
+F 0 "R7" V 2250 6875 50  0000 L CNN
+F 1 "3.3k" V 2100 6850 50  0000 L CNN
+F 2 "Resistors_ThroughHole:R_Axial_DIN0207_L6.3mm_D2.5mm_P2.54mm_Vertical" H 2175 6925 50  0001 C CNN
+F 3 "" H 2175 6925 50  0001 C CNN
+	1    2175 6925
+	0    -1   -1   0
+$EndComp
+Wire Wire Line
+	1950 6925 2075 6925
+Wire Wire Line
+	2075 6675 1950 6675
+Connection ~ 1950 6675
+Wire Wire Line
+	3125 6925 3125 7175
 $EndSCHEMATC

Commit message: Added BDD CPLD code 0.5.1
Changed lines of the file:
@@
 P 3275 6175
 F 0 "#PWR038" H 3275 5925 50  0001 C CNN
-F 1 "GND" H 3275 6025 50  0000 C CNN
+F 1 "GND" V 3275 5975 50  0000 C CNN
 F 2 "" H 3275 6175 50  0001 C CNN
 F 3 "" H 3275 6175 50  0001 C CNN

Commit message: Removed two ram chips, down to 1 MiB.
Parts:
- removed D2, D3: D, Diodes_ThroughHole:D_DO-35_SOD27_P7.62mm_Horizontal, symbol D
- added D2: DIRQ1, Diodes_ThroughHole:D_T-1_P5.08mm_Horizontal, symbol Device:D_Schottky
- added D3: DIRQ2, Diodes_ThroughHole:D_T-1_P5.08mm_Horizontal, symbol Device:D_Schottky
- C16, C17: symbol C_Small -> device:C_Small
- D4: symbol LED -> device:LED
- J3: footprint Connectors_IDC:IDC-Header_2x07_Pitch2.54mm_Straight -> Connectors_IDC:IDC-Header_2x07_Pitch2.54mm_Angled; symbol CONN_02X07 -> conn:CONN_02X07
- J4: footprint Connectors_IDC:IDC-Header_2x20_Pitch2.54mm_Straight -> Connectors_IDC:IDC-Header_2x20_Pitch2.54mm_Angled; symbol CONN_02X20 -> conn:CONN_02X20
- R6: symbol R_Small -> device:R_Small
- R7: value 3.3k -> 470; symbol R_Small -> device:R_Small
- U7, U8: symbol WD65C22PLCC44 -> saturn:WD65C22PLCC44
Connections:
- net ~IRQ: now also D2.2 (A), D3.2 (A); no longer J4.31 (P31)
- net ~IRQVIA1: now reaches U7.23 (~IRQ)
- net ~IRQVIA1: now also D2.1 (K)
- net at U8.23 (~IRQ): now also D3.1 (K)
- no-connect marks 11 -> 12
Other:
- note added: "VIA1 (00:FEC0 - 00:FEDF)"
- note added: "VIA2 (00:FEA0 - 00:FEBF)"
- moved on the sheet: D4, R7
