File: HW/via_and_ide.sch (KiCad schematic (older format))
At the start: 11 parts, among them J3 VIA2PB, J4 IDE, U7 WD65C22PLCC44, U8 WD65C22PLCC44

Commit message: Fixed bus error in RTC design.
Parts:
- C16, C17: symbol device:C_Small -> saturn-rescue:C_Small-device
- D2, D3: symbol Device:D_Schottky -> saturn-rescue:D_Schottky-Device
- D4: symbol device:LED -> saturn-rescue:LED-device
- J3: symbol conn:CONN_02X07 -> saturn-rescue:CONN_02X07-conn
- J4: symbol conn:CONN_02X20 -> saturn-rescue:CONN_02X20-conn
- R6, R7: symbol device:R_Small -> saturn-rescue:R_Small-device
Changed lines of the file:
@@
 EESchema Schematic File Version 4
 LIBS:saturn-cache
-EELAYER 26 0
+EELAYER 29 0
 EELAYER END
 $Descr A4 11693 8268
@@
 $EndComp
 $Comp
-L conn:CONN_02X20 J4
+L saturn-rescue:CONN_02X20-conn J4
 U 1 1 5A3C11DF
 P 4125 6225
@@
 $EndComp
 $Comp
-L conn:CONN_02X07 J3
+L saturn-rescue:CONN_02X07-conn J3
 U 1 1 5A3C12B2
 P 6200 3450
@@
 ~VIA2SEL
 $Comp
-L power1:VCC #PWR036
+L saturn-rescue:VCC-power1 #PWR036
 U 1 1 5A3DECA8
 P 3950 3000
@@
 $EndComp
 $Comp
-L power1:VCC #PWR037
+L saturn-rescue:VCC-power1 #PWR037
 U 1 1 5A3DEEFA
 P 8950 3000
@@
 $EndComp
 $Comp
-L power1:GND #PWR038
+L saturn-rescue:GND-power1 #PWR038
 U 1 1 5A3DF2AF
 P 7950 4625
@@
 $EndComp
 $Comp
-L power1:GND #PWR039
+L saturn-rescue:GND-power1 #PWR039
 U 1 1 5A3DF646
 P 2950 4625
@@
 $EndComp
 $Comp
-L power1:VCC #PWR040
+L saturn-rescue:VCC-power1 #PWR040
 U 1 1 5A3DFA06
 P 7950 875
@@
 $EndComp
 $Comp
-L power1:VCC #PWR041
+L saturn-rescue:VCC-power1 #PWR041
 U 1 1 5A3DFA22
 P 2950 875
@@
 $EndComp
 $Comp
-L device:C_Small C17
+L saturn-rescue:C_Small-device C17
 U 1 1 5A3DFACE
 P 8375 925
@@
 $EndComp
 $Comp
-L device:C_Small C16
+L saturn-rescue:C_Small-device C16
 U 1 1 5A3DFDF6
 P 3275 925
@@
 IDE-D15
 $Comp
-L power1:VCC #PWR042
+L saturn-rescue:VCC-power1 #PWR042
 U 1 1 5A3E3F24
 P 6200 3925
@@
 $EndComp
 $Comp
-L power1:GND #PWR043
+L saturn-rescue:GND-power1 #PWR043
 U 1 1 5A3E3F44
 P 6200 2875
@@
 ~IDE:CS1
 $Comp
-L power1:GND #PWR044
+L saturn-rescue:GND-power1 #PWR044
 U 1 1 5A3E84F7
 P 5175 7250
@@
 IDE-A2
 $Comp
-L power1:GND #PWR045
+L saturn-rescue:GND-power1 #PWR045
 U 1 1 5A3E9E8F
 P 4975 5275
@@
 NoConn ~ 3875 6275
 $Comp
-L power1:GND #PWR046
+L saturn-rescue:GND-power1 #PWR046
 U 1 1 5A3ECBDD
 P 3275 6175
@@
 	9450 3925 9675 3925
 $Comp
-L device:LED D4
+L saturn-rescue:LED-device D4
 U 1 1 5AA70441
 P 2500 7175
@@
 ~IDE:DASP
 $Comp
-L power1:VCC #PWR047
+L saturn-rescue:VCC-power1 #PWR047
 U 1 1 5AA712EE
 P 1950 6475
@@
 $EndComp
 $Comp
-L device:R_Small R6
+L saturn-rescue:R_Small-device R6
 U 1 1 5AA72016
 P 2175 6675
@@
 $EndComp
 $Comp
-L device:R_Small R7
+L saturn-rescue:R_Small-device R7
 U 1 1 5AA72069
 P 2175 7175
@@
 	3650 1750 3950 1750
 $Comp
-L Device:D_Schottky D3
+L saturn-rescue:D_Schottky-Device D3
 U 1 1 5C26C801
 P 9300 3925
@@
 $EndComp
 $Comp
-L Device:D_Schottky D2
+L saturn-rescue:D_Schottky-Device D2
 U 1 1 5C26C9C0
 P 4375 3925

Commit message: Cosmetic changes to schema. Parking this project as router can't find a route.
Parts:
- U7, U8: footprint saturn:PLCC-44_THT-Socket -> Package_LCC:PLCC-44_THT-Socket
Changed lines of the file:
@@
 F 0 "U7" H 2675 3375 60  0000 C CNN
 F 1 "WD65C22PLCC44" V 2950 1600 60  0000 C CNN
-F 2 "saturn:PLCC-44_THT-Socket" H 2375 2325 60  0001 C CNN
+F 2 "Package_LCC:PLCC-44_THT-Socket" H 2375 2325 60  0001 C CNN
 F 3 "" H 2375 2325 60  0000 C CNN
 	1    2875 2300
@@
 F 0 "U8" H 7675 3375 60  0000 C CNN
 F 1 "WD65C22PLCC44" V 7950 1600 60  0000 C CNN
-F 2 "saturn:PLCC-44_THT-Socket" H 7375 2325 60  0001 C CNN
+F 2 "Package_LCC:PLCC-44_THT-Socket" H 7375 2325 60  0001 C CNN
 F 3 "" H 7375 2325 60  0000 C CNN
 	1    7875 2300
