File: HW/controll_logic.sch (KiCad schematic (older format))
At the start: 30 parts, among them J5 POWER_IN, J6 JTAG, J8 Stop System, Q1 DS1813, SW1 RESET, SW2 PANIC, U10 TL7705B, U11 ispMACH4A, U9 74HC74, X2 16MHz

Commit message: Fixed bus error in RTC design.
Parts:
- C14, C18, C19: symbol device:CP_Small -> saturn-rescue:CP_Small-device
- C15, C21, C22: symbol device:C_Small -> saturn-rescue:C_Small-device
- D1: symbol device:LED -> saturn-rescue:LED-device
- F1, F2: symbol device:Fuse -> saturn-rescue:Fuse-device
- H1, H2, H3, H4: symbol Mechanical:MountingHole -> saturn-rescue:MountingHole-Mechanical
- J5: symbol conn:CONN_01X04 -> saturn-rescue:CONN_01X04-conn
- J6: symbol conn:CONN_02X05 -> saturn-rescue:CONN_02X05-conn
- J8: symbol conn:CONN_01X03 -> saturn-rescue:CONN_01X03-conn
- Q1: symbol device:Q_NPN_EBC -> saturn-rescue:Q_NPN_EBC-device
- R1, R2, R3, R4: symbol device:R_Small -> saturn-rescue:R_Small-device
- RN1: symbol device:R_Network08 -> saturn-rescue:R_Network08-device
- RN2: symbol device:R_Network04 -> saturn-rescue:R_Network04-device
- SW1, SW2: symbol switches:SW_Push -> saturn-rescue:SW_Push-switches
- U9: symbol 74xx1:74HC74 -> saturn-rescue:74HC74-74xx1
- X2: symbol Oscillators:CXO_DIP8 -> saturn-rescue:CXO_DIP8-Oscillators
Changed lines of the file:
@@
 EESchema Schematic File Version 4
 LIBS:saturn-cache
-EELAYER 26 0
+EELAYER 29 0
 EELAYER END
 $Descr A4 11693 8268
@@
 $EndComp
 $Comp
-L 74xx1:74HC74 U9
+L saturn-rescue:74HC74-74xx1 U9
 U 2 1 5A3B42E3
 P 1300 6625
@@
 $EndComp
 $Comp
-L 74xx1:74HC74 U9
+L saturn-rescue:74HC74-74xx1 U9
 U 1 1 5A3B432C
 P 3825 6625
@@
 $EndComp
 $Comp
-L Oscillators:CXO_DIP8 X2
+L saturn-rescue:CXO_DIP8-Oscillators X2
 U 1 1 5A3B45C3
 P 2650 6625
@@
 $EndComp
 $Comp
-L power1:VCC #PWR048
+L saturn-rescue:VCC-power1 #PWR048
 U 1 1 5A3B5086
 P 2650 6075
@@
 $EndComp
 $Comp
-L power1:GND #PWR049
+L saturn-rescue:GND-power1 #PWR049
 U 1 1 5A3B5184
 P 2650 7050
@@
 $EndComp
 $Comp
-L power1:GND #PWR050
+L saturn-rescue:GND-power1 #PWR050
 U 1 1 5A3B51A8
 P 700 7375
@@
 NoConn ~ 1900 6825
 $Comp
-L power1:VCC #PWR051
+L saturn-rescue:VCC-power1 #PWR051
 U 1 1 5A3B65BD
 P 3925 1150
@@
 RES
 $Comp
-L device:C_Small C15
+L saturn-rescue:C_Small-device C15
 U 1 1 5A3B6A11
 P 3925 3650
@@
 $EndComp
 $Comp
-L device:R_Small R3
+L saturn-rescue:R_Small-device R3
 U 1 1 5A3B6A86
 P 4250 3475
@@
 $EndComp
 $Comp
-L device:R_Small R2
+L saturn-rescue:R_Small-device R2
 U 1 1 5A3B6C94
 P 2325 3475
@@
 $EndComp
 $Comp
-L device:CP_Small C14
+L saturn-rescue:CP_Small-device C14
 U 1 1 5A3B6D16
 P 2325 3750
@@
 $EndComp
 $Comp
-L device:R_Small R1
+L saturn-rescue:R_Small-device R1
 U 1 1 5A3B6D93
 P 2000 2950
@@
 $EndComp
 $Comp
-L switches:SW_Push SW1
+L saturn-rescue:SW_Push-switches SW1
 U 1 1 5A3B9114
 P 2000 3375
@@
 $EndComp
 $Comp
-L power1:GND #PWR052
+L saturn-rescue:GND-power1 #PWR052
 U 1 1 5A3B95EF
 P 3125 3850
@@
 $EndComp
 $Comp
-L power1:VCC #PWR053
+L saturn-rescue:VCC-power1 #PWR053
 U 1 1 5A3B9B69
 P 2325 2500
@@
 ~ABT
 $Comp
-L device:R_Network08 RN1
+L saturn-rescue:R_Network08-device RN1
 U 1 1 5A416FA2
 P 4325 1550
@@
 $EndComp
 $Comp
-L device:Fuse F2
+L saturn-rescue:Fuse-device F2
 U 1 1 5A43A547
 P 9525 5000
@@
 $EndComp
 $Comp
-L device:Fuse F1
+L saturn-rescue:Fuse-device F1
 U 1 1 5A43A5A2
 P 8350 5350
@@
 $EndComp
 $Comp
-L conn:CONN_01X04 J5
+L saturn-rescue:CONN_01X04-conn J5
 U 1 1 5A43C29B
 P 10300 5250
@@
 $EndComp
 $Comp
-L device:CP_Small C19
+L saturn-rescue:CP_Small-device C19
 U 1 1 5A43C8E4
 P 9350 5300
@@
 $EndComp
 $Comp
-L device:CP_Small C18
+L saturn-rescue:CP_Small-device C18
 U 1 1 5A43C96F
 P 7950 5575
@@
 $EndComp
 $Comp
-L device:LED D1
+L saturn-rescue:LED-device D1
 U 1 1 5A43C9AA
 P 8725 5575
@@
 $EndComp
 $Comp
-L device:R_Small R4
+L saturn-rescue:R_Small-device R4
 U 1 1 5A43CA45
 P 8725 5225
@@
 $EndComp
 $Comp
-L power1:PWR_FLAG #FLG054
+L saturn-rescue:PWR_FLAG-power1 #FLG054
 U 1 1 5A43CDBE
 P 10100 5000
@@
 $EndComp
 $Comp
-L power1:PWR_FLAG #FLG055
+L saturn-rescue:PWR_FLAG-power1 #FLG055
 U 1 1 5A43CDFA
 P 10000 5825
@@
 NoConn ~ 9175 5100
 $Comp
-L power1:GND #PWR056
+L saturn-rescue:GND-power1 #PWR056
 U 1 1 5A43D8F9
 P 7050 5825
@@
 $EndComp
 $Comp
-L power1:VCC #PWR057
+L saturn-rescue:VCC-power1 #PWR057
 U 1 1 5A43D935
 P 7600 5050
@@
 $EndComp
 $Comp
-L power1:+5V #PWR058
+L saturn-rescue:+5V-power1 #PWR058
 U 1 1 5A43F37E
 P 7600 5350
@@
 $EndComp
 $Comp
-L conn:CONN_02X05 J6
+L saturn-rescue:CONN_02X05-conn J6
 U 1 1 5A4410D6
 P 6250 5350
@@
 TDO
 $Comp
-L device:C_Small C22
+L saturn-rescue:C_Small-device C22
 U 1 1 5A449952
 P 8675 1075
@@
 $EndComp
 $Comp
-L device:C_Small C21
+L saturn-rescue:C_Small-device C21
 U 1 1 5A449A79
 P 7850 1075
@@
 $EndComp
 $Comp
-L power1:GND #PWR060
+L saturn-rescue:GND-power1 #PWR060
 U 1 1 5A44C14E
 P 8300 4600
@@
 STP
 $Comp
-L conn:CONN_01X03 J8
+L saturn-rescue:CONN_01X03-conn J8
 U 1 1 5AA76556
 P 4750 4875
@@
 RDY
 $Comp
-L power1:GND #PWR061
+L saturn-rescue:GND-power1 #PWR061
 U 1 1 5AA76AFA
 P 4275 4975
@@
 $EndComp
 $Comp
-L power1:PWR_FLAG #FLG062
+L saturn-rescue:PWR_FLAG-power1 #FLG062
 U 1 1 5AA7AD12
 P 7875 5050
@@
 $EndComp
 $Comp
-L power1:PWR_FLAG #FLG063
+L saturn-rescue:PWR_FLAG-power1 #FLG063
 U 1 1 5AA7AE0B
 P 7950 5350
@@
 $EndComp
 $Comp
-L power1:VCC #PWR064
+L saturn-rescue:VCC-power1 #PWR064
 U 1 1 5AA1B8B6
 P 8225 1075
@@
 $EndComp
 $Comp
-L power1:VCC #PWR065
+L saturn-rescue:VCC-power1 #PWR065
 U 1 1 5AA1B8FA
 P 8325 1075
@@
 $EndComp
 $Comp
-L device:Q_NPN_EBC Q1
+L saturn-rescue:Q_NPN_EBC-device Q1
 U 1 1 5B5CB0CA
 P 2750 4950
@@
 ~NMI
 $Comp
-L power1:GND #PWR066
+L saturn-rescue:GND-power1 #PWR066
 U 1 1 5B5CB6C5
 P 2650 5325
@@
 $EndComp
 $Comp
-L power1:VCC #PWR067
+L saturn-rescue:VCC-power1 #PWR067
 U 1 1 5B5CB70D
 P 2950 4950
@@
 $EndComp
 $Comp
-L switches:SW_Push SW2
+L saturn-rescue:SW_Push-switches SW2
 U 1 1 5B5CB858
 P 2150 5025
@@
 Connection ~ 2650 5325
 $Comp
-L power:VCC #PWR055
+L saturn-rescue:VCC-power #PWR055
 U 1 1 5BF4F6F5
 P 5600 4300
@@
 	8300 4450 8350 4450
 $Comp
-L power:GND #PWR0105
+L saturn-rescue:GND-power #PWR0105
 U 1 1 5C21E5C0
 P 8450 4600
@@
 $EndComp
 $Comp
-L power:GND #PWR0106
+L saturn-rescue:GND-power #PWR0106
 U 1 1 5C21E832
 P 8100 4600
@@
 Connection ~ 8100 4450
 $Comp
-L Mechanical:MountingHole H1
+L saturn-rescue:MountingHole-Mechanical H1
 U 1 1 5C2392E9
 P 5650 6075
@@
 $EndComp
 $Comp
-L Mechanical:MountingHole H2
+L saturn-rescue:MountingHole-Mechanical H2
 U 1 1 5C239368
 P 5650 6300
@@
 $EndComp
 $Comp
-L Mechanical:MountingHole H3
+L saturn-rescue:MountingHole-Mechanical H3
 U 1 1 5C2393BC
 P 5650 6550
@@
 $EndComp
 $Comp
-L Mechanical:MountingHole H4
+L saturn-rescue:MountingHole-Mechanical H4
 U 1 1 5C9ECC4F
 P 5650 6800
@@
 $EndComp
 $Comp
-L device:R_Network04 RN2
+L saturn-rescue:R_Network04-device RN2
 U 1 1 5C9EDD0C
 P 5800 4700

Commit message: Cosmetic changes to schema. Parking this project as router can't find a route.
Parts:
- U11: footprint saturn:PLCC-44_THT-Socket -> Package_LCC:PLCC-44_THT-Socket
Changed lines of the file:
@@
 F 0 "U11" H 8275 3775 60  0000 C CNN
 F 1 "ispMACH4A" V 8275 1950 60  0000 C CNN
-F 2 "saturn:PLCC-44_THT-Socket" H 7950 2300 60  0001 C CNN
+F 2 "Package_LCC:PLCC-44_THT-Socket" H 7950 2300 60  0001 C CNN
 F 3 "" H 7950 2300 60  0001 C CNN
 	1    8275 2325
