File: HW/duart_line_drivers.sch (KiCad schematic (older format))
At the start: 12 parts, among them J1 RS232a, J2 RS232b, U3 MAX238, U4 SC28L92PLCC44, X1 3.6864 MHz

Commit message: Fixed bus error in RTC design.
Parts:
- C1, C2, C3, C4, C5: symbol device:CP_Small -> saturn-rescue:CP_Small-device
- C6: symbol device:C -> saturn-rescue:C-device
- R5: symbol device:R_Small -> saturn-rescue:R_Small-device
- X1: symbol Oscillators:CXO_DIP8 -> saturn-rescue:CXO_DIP8-Oscillators
Changed lines of the file:
@@
 EESchema Schematic File Version 4
 LIBS:saturn-cache
-EELAYER 26 0
+EELAYER 29 0
 EELAYER END
 $Descr A4 11693 8268
@@
 $EndComp
 $Comp
-L device:CP_Small C4
+L saturn-rescue:CP_Small-device C4
 U 1 1 5A14E4E1
 P 5000 1825
@@
 $EndComp
 $Comp
-L device:CP_Small C5
+L saturn-rescue:CP_Small-device C5
 U 1 1 5A14E779
 P 5000 2225
@@
 $EndComp
 $Comp
-L device:CP_Small C1
+L saturn-rescue:CP_Small-device C1
 U 1 1 5A14E8FA
 P 3125 1450
@@
 $EndComp
 $Comp
-L power1:VCC #PWR025
+L saturn-rescue:VCC-power1 #PWR025
 U 1 1 5A14EA51
 P 4025 1225
@@
 $EndComp
 $Comp
-L device:CP_Small C3
+L saturn-rescue:CP_Small-device C3
 U 1 1 5A14EA93
 P 4850 1350
@@
 $EndComp
 $Comp
-L power1:GND #PWR026
+L saturn-rescue:GND-power1 #PWR026
 U 1 1 5A14EB59
 P 5075 1350
@@
 $EndComp
 $Comp
-L device:CP_Small C2
+L saturn-rescue:CP_Small-device C2
 U 1 1 5A14F3DD
 P 3125 2125
@@
 $EndComp
 $Comp
-L power1:GND #PWR027
+L saturn-rescue:GND-power1 #PWR027
 U 1 1 5A14F46D
 P 3125 2225
@@
 $EndComp
 $Comp
-L power1:GND #PWR028
+L saturn-rescue:GND-power1 #PWR028
 U 1 1 5A14F656
 P 4025 4450
@@
 RS232CTSb
 $Comp
-L power1:GND #PWR029
+L saturn-rescue:GND-power1 #PWR029
 U 1 1 5A1536E4
 P 1150 3725
@@
 $EndComp
 $Comp
-L power1:GND #PWR030
+L saturn-rescue:GND-power1 #PWR030
 U 1 1 5A153732
 P 1150 3000
@@
 NoConn ~ 6200 4150
 $Comp
-L Oscillators:CXO_DIP8 X1
+L saturn-rescue:CXO_DIP8-Oscillators X1
 U 1 1 5A156C53
 P 8650 4250
@@
 $EndComp
 $Comp
-L power1:VCC #PWR031
+L saturn-rescue:VCC-power1 #PWR031
 U 1 1 5A1570C4
 P 8650 3950
@@
 $EndComp
 $Comp
-L power1:GND #PWR032
+L saturn-rescue:GND-power1 #PWR032
 U 1 1 5A157100
 P 8650 4550
@@
 NoConn ~ 7400 4375
 $Comp
-L power1:VCC #PWR033
+L saturn-rescue:VCC-power1 #PWR033
 U 1 1 5A157C4F
 P 7800 4500
@@
 $EndComp
 $Comp
-L power1:GND #PWR034
+L saturn-rescue:GND-power1 #PWR034
 U 1 1 5A157EAF
 P 6825 5325
@@
 $EndComp
 $Comp
-L device:C C6
+L saturn-rescue:C-device C6
 U 1 1 5A157F44
 P 7650 5325
@@
 ~DUARTSEL
 $Comp
-L device:R_Small R5
+L saturn-rescue:R_Small-device R5
 U 1 1 5A984B90
 P 8225 4050
@@
 A3
 $Comp
-L power1:VCC #PWR035
+L saturn-rescue:VCC-power1 #PWR035
 U 1 1 5AA1B80C
 P 6825 1150
@@
 	8225 4250 8350 4250
 NoConn ~ 4575 3850
+Text Notes 7200 1000 0    60   ~ 12
+DUART (00:FEE0 - 00:FEFF)
 Wire Bus Line
 	7775 2850 7775 3225
 Wire Bus Line
 	7775 1475 7775 2525
-Text Notes 7200 1000 0    60   ~ 12
-DUART (00:FEE0 - 00:FEFF)
 $EndSCHEMATC

Commit message: Cosmetic changes to schema. Parking this project as router can't find a route.
Parts:
- U4: footprint saturn:PLCC-44_THT-Socket -> Package_LCC:PLCC-44_THT-Socket
Changed lines of the file:
@@
 F 0 "U4" H 7125 3625 60  0000 C CNN
 F 1 "SC28L92PLCC44" V 6825 2050 60  0000 C CNN
-F 2 "saturn:PLCC-44_THT-Socket" H 6825 2600 60  0001 C CNN
+F 2 "Package_LCC:PLCC-44_THT-Socket" H 6825 2600 60  0001 C CNN
 F 3 "" H 6825 2600 60  0001 C CNN
 	1    6725 2600
