File: HW/rtc.sch (KiCad schematic (older format))
At the start: 2 parts

Commit message: Simulation of address decoding.
Parts:
- gave numbers to parts that had none: 2
Connections:
- net labels added: A[0..19]
- net labels removed: A[0..18]
Changed lines of the file:
@@
 $EndDescr
 $Comp
-L DS1511Y+ U?
+L DS1511Y+ U12
 U 1 1 5A3D8313
 P 4700 2975
-F 0 "U?" H 4800 3700 60  0000 C CNN
+F 0 "U12" H 4800 3700 60  0000 C CNN
 F 1 "DS1511Y+" V 4750 2975 60  0000 C CNN
 F 2 "" H 4450 3425 60  0001 C CNN
@@
 	3825 1800 3075 1800
 Text Label 3075 1800 0    60   ~ 0
-A[0..18]
+A[0..19]
 Wire Bus Line
 	5675 1800 5675 3000
@@
 D[0..7]
 Text HLabel 3075 1800 0    60   Input ~ 0
-A[0..18]
+A[0..19]
 Text HLabel 5575 3225 2    60   Output ~ 0
 ~PWR
@@
 Connection ~ 4725 3975
 $Comp
-L GND #PWR?
+L GND #PWR36
 U 1 1 5A3D88A1
 P 4725 4175
-F 0 "#PWR?" H 4725 3925 50  0001 C CNN
+F 0 "#PWR36" H 4725 3925 50  0001 C CNN
 F 1 "GND" H 4725 4025 50  0000 C CNN
 F 2 "" H 4725 4175 50  0001 C CNN
@@
 	4725 2100 4725 1875
 $Comp
-L VCC #PWR?
+L VCC #PWR35
 U 1 1 5A3D896E
 P 4725 1875
-F 0 "#PWR?" H 4725 1725 50  0001 C CNN
+F 0 "#PWR35" H 4725 1725 50  0001 C CNN
 F 1 "VCC" H 4725 2025 50  0000 C CNN
 F 2 "" H 4725 1875 50  0001 C CNN
@@
 $EndComp
 $Comp
-L C_Small C?
+L C_Small C20
 U 1 1 5A3D89E9
 P 5025 1925
-F 0 "C?" V 4925 1875 50  0000 L CNN
+F 0 "C20" V 4925 1875 50  0000 L CNN
 F 1 "0.1uF" V 5125 1825 50  0000 L CNN
 F 2 "" H 5025 1925 50  0001 C CNN
@@
 NoConn ~ 5275 3475
 $Comp
-L GND #PWR?
+L GND #PWR37
 U 1 1 5A3DA9B9
 P 5575 3600
-F 0 "#PWR?" H 5575 3350 50  0001 C CNN
+F 0 "#PWR37" H 5575 3350 50  0001 C CNN
 F 1 "GND" H 5575 3450 50  0000 C CNN
 F 2 "" H 5575 3600 50  0001 C CNN

Commit message: ABEL code passes compilation, no tests though. Small changes to schema
Parts:
- C20: footprint (none) -> Capacitors_ThroughHole:C_Disc_D4.7mm_W2.5mm_P5.00mm
- U12: footprint (none) -> Housings_DIP:DIP-28_W15.24mm_Socket
Connections:
- net labels added: A[0..18], ~RES
- net labels removed: A[0..19], ~RST
Changed lines of the file:
@@
 $Descr A4 11693 8268
 encoding utf-8
-Sheet 6 6
+Sheet 6 7
 Title ""
-Date "2017-12-23"
+Date "2018-01-17"
 Rev "0.1"
 Comp "Linux Grotto"
@@
 F 0 "U12" H 4800 3700 60  0000 C CNN
 F 1 "DS1511Y+" V 4750 2975 60  0000 C CNN
-F 2 "" H 4450 3425 60  0001 C CNN
+F 2 "Housings_DIP:DIP-28_W15.24mm_Socket" H 4450 3425 60  0001 C CNN
 F 3 "" H 4450 3425 60  0001 C CNN
 	1    4700 2975
@@
 	3825 1800 3075 1800
 Text Label 3075 1800 0    60   ~ 0
-A[0..19]
+A[0..18]
 Wire Bus Line
 	5675 1800 5675 3000
@@
 D[0..7]
 Text HLabel 3075 1800 0    60   Input ~ 0
-A[0..19]
+A[0..18]
 Text HLabel 5575 3225 2    60   Output ~ 0
 ~PWR
@@
 ~IRQ
 Text HLabel 3925 3575 0    60   Output ~ 0
-~RST
+~RES
 Wire Wire Line
 	5275 3225 5575 3225
@@
 Connection ~ 4725 3975
 $Comp
-L GND #PWR36
+L GND #PWR058
 U 1 1 5A3D88A1
 P 4725 4175
-F 0 "#PWR36" H 4725 3925 50  0001 C CNN
+F 0 "#PWR058" H 4725 3925 50  0001 C CNN
 F 1 "GND" H 4725 4025 50  0000 C CNN
 F 2 "" H 4725 4175 50  0001 C CNN
@@
 	4725 2100 4725 1875
 $Comp
-L VCC #PWR35
+L VCC #PWR059
 U 1 1 5A3D896E
 P 4725 1875
-F 0 "#PWR35" H 4725 1725 50  0001 C CNN
+F 0 "#PWR059" H 4725 1725 50  0001 C CNN
 F 1 "VCC" H 4725 2025 50  0000 C CNN
 F 2 "" H 4725 1875 50  0001 C CNN
@@
 F 0 "C20" V 4925 1875 50  0000 L CNN
 F 1 "0.1uF" V 5125 1825 50  0000 L CNN
-F 2 "" H 5025 1925 50  0001 C CNN
+F 2 "Capacitors_ThroughHole:C_Disc_D4.7mm_W2.5mm_P5.00mm" H 5025 1925 50  0001 C CNN
 F 3 "" H 5025 1925 50  0001 C CNN
 	1    5025 1925
@@
 NoConn ~ 5275 3475
 $Comp
-L GND #PWR37
+L GND #PWR060
 U 1 1 5A3DA9B9
 P 5575 3600
-F 0 "#PWR37" H 5575 3350 50  0001 C CNN
+F 0 "#PWR060" H 5575 3350 50  0001 C CNN
 F 1 "GND" H 5575 3450 50  0000 C CNN
 F 2 "" H 5575 3600 50  0001 C CNN

Commit message: Removed two ram chips, down to 1 MiB.
Parts:
- added J7: Expansion Bus, Connectors_IDC:IDC-Header_2x20_Pitch2.54mm_Angled, symbol conn:CONN_02X20
- C20: symbol C_Small -> device:C_Small
- U12: symbol DS1511Y+ -> saturn:DS1511Y+
Connections:
- net labels added: A10, A11, A12, A13, A14, A15, A5, A6, A7, A8, A9, CLK, R/~W, RDY, ~IOSEL2, ~IOSEL3, ~NMI
- wire segments 28 -> 74
- no-connect marks 1 -> 3
Other:
- note added: "IOSEL2 (00:FE60 - 00:FE7F)"
- note added: "IOSEL3 (00:FE40 - 00:FE5F)"
- note added: "RTC (00:FE80 - 00:FE9F)"

Commit message: Added new footprints. Added docs
Parts:
- J7: footprint Connectors_IDC:IDC-Header_2x20_Pitch2.54mm_Angled -> Connectors_IDC:IDC-Header_2x20_Pitch2.54mm_Straight
Changed lines of the file:
@@
 F 0 "J7" H 9525 3850 50  0000 C CNN
 F 1 "Expansion Bus" H 9475 1450 50  0000 C CNN
-F 2 "Connectors_IDC:IDC-Header_2x20_Pitch2.54mm_Angled" H 9450 1850 50  0001 C CNN
+F 2 "Connectors_IDC:IDC-Header_2x20_Pitch2.54mm_Straight" H 9450 1850 50  0001 C CNN
 F 3 "" H 9450 1850 50  0001 C CNN
 	1    9450 2800

Commit message: Fixed bus error in RTC design.
Parts:
- C20: symbol device:C_Small -> saturn-rescue:C_Small-device
- J7: symbol conn:CONN_02X20 -> saturn-rescue:CONN_02X20-conn
Changed lines of the file:
@@
 EESchema Schematic File Version 4
 LIBS:saturn-cache
-EELAYER 26 0
+EELAYER 29 0
 EELAYER END
 $Descr A4 11693 8268
@@
 Connection ~ 4725 3975
 $Comp
-L power1:GND #PWR068
+L saturn-rescue:GND-power1 #PWR068
 U 1 1 5A3D88A1
 P 4725 4175
@@
 	4725 2100 4725 1925
 $Comp
-L power1:VCC #PWR069
+L saturn-rescue:VCC-power1 #PWR069
 U 1 1 5A3D896E
 P 4725 1875
@@
 $EndComp
 $Comp
-L device:C_Small C20
+L saturn-rescue:C_Small-device C20
 U 1 1 5A3D89E9
 P 5025 1925
@@
 NoConn ~ 5275 3475
 $Comp
-L power1:GND #PWR070
+L saturn-rescue:GND-power1 #PWR070
 U 1 1 5A3DA9B9
 P 5575 3600
@@
 	4725 4150 4725 4175
 $Comp
-L power:VCC #PWR0101
+L saturn-rescue:VCC-power #PWR0101
 U 1 1 5BE1F817
 P 9450 1700
@@
 $EndComp
 $Comp
-L power:GND #PWR0102
+L saturn-rescue:GND-power #PWR0102
 U 1 1 5BE1F849
 P 9450 3900
@@
 Wire Wire Line
 	9700 3350 10000 3350
-Wire Wire Line
-	9700 3450 10000 3450
 Wire Wire Line
 	9700 3550 10000 3550
@@
 Text Label 10000 3350 2    50   ~ 0
 A14
-Text Label 10000 3450 2    50   ~ 0
-A15
-Entry Bus Bus
-	8800 1850 8900 1950
-Entry Bus Bus
-	8800 1950 8900 2050
-Entry Bus Bus
-	8800 2050 8900 2150
-Entry Bus Bus
-	8800 2150 8900 2250
-Entry Bus Bus
-	8800 2250 8900 2350
-Entry Bus Bus
-	8800 2350 8900 2450
-Entry Bus Bus
-	8800 2450 8900 2550
-Entry Bus Bus
-	8800 2550 8900 2650
-Entry Bus Bus
-	10000 1950 10100 1850
-Entry Bus Bus
-	10000 2050 10100 1950
-Entry Bus Bus
-	10000 2150 10100 2050
-Entry Bus Bus
-	10000 2250 10100 2150
-Entry Bus Bus
-	10000 2350 10100 2250
-Entry Bus Bus
-	10000 2450 10100 2350
-Entry Bus Bus
-	10000 2550 10100 2450
-Entry Bus Bus
-	10000 2650 10100 2550
-Entry Bus Bus
-	10000 2750 10100 2650
-Entry Bus Bus
-	10000 2850 10100 2750
-Entry Bus Bus
-	10000 2950 10100 2850
-Entry Bus Bus
-	10000 3050 10100 2950
-Entry Bus Bus
-	10000 3150 10100 3050
-Entry Bus Bus
-	10000 3250 10100 3150
-Entry Bus Bus
-	10000 3350 10100 3250
-Entry Bus Bus
-	10000 3450 10100 3350
 Wire Bus Line
 	8800 1850 8225 1850
@@
 NoConn ~ 9200 2750
 $Comp
-L conn:CONN_02X20 J7
+L saturn-rescue:CONN_02X20-conn J7
 U 1 1 5BE1F74C
 P 9450 2800
@@
 Wire Wire Line
 	9200 3250 8900 3250
-Wire Bus Line
-	3825 1800 3825 2700
-Wire Bus Line
-	8800 1850 8800 2550
-Wire Bus Line
-	5675 1800 5675 3000
-Wire Bus Line
-	10100 1850 10100 3350
 Text Notes 8800 4400 0    60   ~ 12
 IOSEL2 (00:FE60 - 00:FE7F)
 Text Notes 8800 4525 0    60   ~ 12
 IOSEL3 (00:FE40 - 00:FE5F)
+Wire Wire Line
+	9700 3450 10000 3450
+Text Label 10000 3450 2    50   ~ 0
+A15
+Wire Bus Line
+	10100 1850 10100 3350
+Wire Bus Line
+	8800 1850 8800 2550
+Wire Bus Line
+	3825 1800 3825 2700
+Wire Bus Line
+	5675 1800 5675 3000
+Entry Wire Line
+	8800 1850 8900 1950
+Entry Wire Line
+	8800 1950 8900 2050
+Entry Wire Line
+	8800 2050 8900 2150
+Entry Wire Line
+	8800 2150 8900 2250
+Entry Wire Line
+	8800 2250 8900 2350
+Entry Wire Line
+	8800 2350 8900 2450
+Entry Wire Line
+	8800 2450 8900 2550
+Entry Wire Line
+	8800 2550 8900 2650
+Entry Wire Line
+	10000 1950 10100 1850
+Entry Wire Line
+	10000 2050 10100 1950
+Entry Wire Line
+	10000 2150 10100 2050
+Entry Wire Line
+	10000 2250 10100 2150
+Entry Wire Line
+	10000 2350 10100 2250
+Entry Wire Line
+	10000 2450 10100 2350
+Entry Wire Line
+	10000 2550 10100 2450
+Entry Wire Line
+	10000 2650 10100 2550
+Entry Wire Line
+	10000 2750 10100 2650
+Entry Wire Line
+	10000 2850 10100 2750
+Entry Wire Line
+	10000 2950 10100 2850
+Entry Wire Line
+	10000 3050 10100 2950
+Entry Wire Line
+	10000 3150 10100 3050
+Entry Wire Line
+	10000 3250 10100 3150
+Entry Wire Line
+	10000 3350 10100 3250
+Entry Wire Line
+	10000 3450 10100 3350
 $EndSCHEMATC
