File: HW/saturn.kicad_pcb (KiCad board)
At the start: 4 copper layers, 0 parts

Commit message: Removed two ram chips, down to 1 MiB.
Parts:
- added C1: 1.0uF, Capacitors_ThroughHole:CP_Radial_Tantal_D4.5mm_P2.50mm, F.Cu at (169.2, 51.3)
- added C10: 0.1uF, Capacitors_ThroughHole:C_Disc_D4.7mm_W2.5mm_P5.00mm, F.Cu at (56.4, 82.8)
- added C11: 0.1uF, Capacitors_ThroughHole:C_Disc_D4.7mm_W2.5mm_P5.00mm, F.Cu at (78.2, 60.5)
- added C12: 0.1uF, Capacitors_ThroughHole:C_Disc_D4.7mm_W2.5mm_P5.00mm, F.Cu at (49.8, 61.0)
- added C13: 0.1uF, Capacitors_ThroughHole:C_Disc_D4.7mm_W2.5mm_P5.00mm, F.Cu at (82.8, 82.8)
- added C14: 15uF, Capacitors_ThroughHole:CP_Radial_D5.0mm_P2.50mm, F.Cu at (171.2, 126.5)
- added C15: 0.1uF, Capacitors_ThroughHole:C_Disc_D4.7mm_W2.5mm_P5.00mm, F.Cu at (173.2, 55.4)
- added C16: 0.1uF, Capacitors_ThroughHole:C_Disc_D4.7mm_W2.5mm_P5.00mm, F.Cu at (67.1, 51.3)
- added C17: 0.1uF, Capacitors_ThroughHole:C_Disc_D4.7mm_W2.5mm_P5.00mm, F.Cu at (94.0, 43.7)
- added C18: 100uF, Capacitors_ThroughHole:CP_Radial_D6.3mm_P2.50mm, F.Cu at (201.7, 51.8)
- added C19: 100uF, Capacitors_ThroughHole:CP_Radial_D6.3mm_P2.50mm, F.Cu at (182.4, 37.6)
- added C2: 1.0uF, Capacitors_ThroughHole:CP_Radial_Tantal_D4.5mm_P2.50mm, F.Cu at (168.7, 33.5)
- added C20: 0.1uF, Capacitors_ThroughHole:C_Disc_D4.7mm_W2.5mm_P5.00mm, F.Cu at (99.6, 120.4)
- added C21: 0.1uF, Capacitors_ThroughHole:C_Disc_D4.7mm_W2.5mm_P5.00mm, F.Cu at (49.8, 55.9)
- added C22: 0.1uF, Capacitors_ThroughHole:C_Disc_D4.7mm_W2.5mm_P5.00mm, F.Cu at (67.1, 31.5)
- added C23: 0.1uF, Capacitors_ThroughHole:C_Disc_D4.7mm_W2.5mm_P5.00mm, F.Cu at (131.6, 60.5)
- added C24: 0.1uF, Capacitors_ThroughHole:C_Disc_D4.7mm_W2.5mm_P5.00mm, F.Cu at (132.1, 82.8)
- added C25: 0.1uF, Capacitors_ThroughHole:C_Disc_D4.7mm_W2.5mm_P5.00mm, F.Cu at (109.7, 82.8)
- added C26: 0.1uF, Capacitors_ThroughHole:C_Disc_D4.7mm_W2.5mm_P5.00mm, F.Cu at (109.7, 60.5)
- added C3: 1.0uF, Capacitors_ThroughHole:CP_Radial_Tantal_D4.5mm_P2.50mm, F.Cu at (163.1, 51.3)
- added C4: 1.0uF, Capacitors_ThroughHole:CP_Radial_Tantal_D4.5mm_P2.50mm, F.Cu at (174.2, 51.3)
- added C5: 1.0uF, Capacitors_ThroughHole:CP_Radial_Tantal_D4.5mm_P2.50mm, F.Cu at (176.2, 34.5)
- added C6: 0.1uF, Capacitors_ThroughHole:C_Disc_D4.7mm_W2.5mm_P5.00mm, F.Cu at (65.0, 112.3)
- added C7: 0.1uF, Capacitors_ThroughHole:C_Disc_D4.7mm_W2.5mm_P5.00mm, F.Cu at (23.9, 55.9)
- added C8: 0.1uF, Capacitors_ThroughHole:C_Disc_D4.7mm_W2.5mm_P5.00mm, F.Cu at (23.9, 29.0)
- added C9: 0.1uF, Capacitors_ThroughHole:C_Disc_D4.7mm_W2.5mm_P5.00mm, F.Cu at (22.4, 84.8)
- added D1: LED, LEDs:LED_D3.0mm, F.Cu at (188.0, 51.8)
- added D2: DIRQ1, Diodes_ThroughHole:D_T-1_P5.08mm_Horizontal, F.Cu at (114.3, 57.4)
- added D3: DIRQ2, Diodes_ThroughHole:D_T-1_P5.08mm_Horizontal, F.Cu at (85.9, 56.9)
- added D4: LED, LEDs:LED_D3.0mm, F.Cu at (188.5, 44.2)
- added F1: 200mA, Fuse_Holders_and_Fuses:Fuseholder5x20_horiz_open_Schurter_0031_8201, F.Cu at (199.1, 43.7)
- added F2: 1A, Fuse_Holders_and_Fuses:Fuseholder5x20_horiz_open_Schurter_0031_8201, F.Cu at (221.5, 33.0)
- added H1: MountingHole, Mounting_Holes:MountingHole_3.2mm_M3_DIN965_Pad, F.Cu at (18.8, 18.8)
- added H2: MountingHole, Mounting_Holes:MountingHole_3.2mm_M3_DIN965_Pad, F.Cu at (23.4, 148.3)
- added H3: MountingHole, Mounting_Holes:MountingHole_3.2mm_M3_DIN965_Pad, F.Cu at (217.9, 19.8)
- added H4: MountingHole, Mounting_Holes:MountingHole_3.2mm_M3_DIN965_Pad, F.Cu at (213.9, 143.3)
- added J1: RS232a, Connectors_IDC:IDC-Header_2x05_Pitch2.54mm_Angled, F.Cu at (176.8, 29.0)
- added J2: RS232b, Connectors_IDC:IDC-Header_2x05_Pitch2.54mm_Angled, F.Cu at (154.4, 29.0)
- added J3: VIA2PB, Connectors_IDC:IDC-Header_2x07_Pitch2.54mm_Angled, F.Cu at (77.2, 90.9)
- added J4: IDE, Connectors_IDC:IDC-Header_2x20_Pitch2.54mm_Angled, F.Cu at (94.0, 29.0)
- added J5: POWER_IN, Connectors_Molex:Molex_NanoFit_1x04x2.50mm_Angled, F.Cu at (204.7, 25.9)
- added J6: JTAG, Connectors_IDC:IDC-Header_2x05_Pitch2.54mm_Straight, F.Cu at (19.3, 63.5)
- added J7: Expansion Bus, Connectors_IDC:IDC-Header_2x20_Pitch2.54mm_Angled, F.Cu at (27.4, 29.0)
- added J8: Stop System, Pin_Headers:Pin_Header_Straight_1x03_Pitch2.54mm, F.Cu at (141.7, 140.2)
- added JP1: Enable ISP, Pin_Headers:Pin_Header_Straight_1x02_Pitch2.54mm, F.Cu at (19.3, 80.8)
- added Q1: DS1813, TO_SOT_Packages_THT:TO-92_Inline_Narrow_Oval, F.Cu at (69.1, 120.9)
- added R1: 22k, Resistors_ThroughHole:R_Axial_DIN0207_L6.3mm_D2.5mm_P2.54mm_Vertical, F.Cu at (78.2, 113.8)
- added R2: 475, Resistors_ThroughHole:R_Axial_DIN0207_L6.3mm_D2.5mm_P2.54mm_Vertical, F.Cu at (169.7, 120.9)
- added R3: 3.3k, Resistors_ThroughHole:R_Axial_DIN0207_L6.3mm_D2.5mm_P2.54mm_Vertical, F.Cu at (177.8, 132.1)
- added R4: 470, Resistors_ThroughHole:R_Axial_DIN0207_L6.3mm_D2.5mm_P2.54mm_Vertical, F.Cu at (180.8, 56.4)
- added R5: 470, Resistors_ThroughHole:R_Axial_DIN0207_L6.3mm_D2.5mm_P2.54mm_Vertical, F.Cu at (138.2, 135.1)
- added R6: 3.3k, Resistors_ThroughHole:R_Axial_DIN0207_L6.3mm_D2.5mm_P2.54mm_Vertical, F.Cu at (153.4, 52.3)
- added R7: 470, Resistors_ThroughHole:R_Axial_DIN0207_L6.3mm_D2.5mm_P2.54mm_Vertical, F.Cu at (148.8, 34.0)
- added RN1: 3.3k, Resistors_THT:R_Array_SIP9, F.Cu at (165.6, 120.9)
- added RN2: 3.3k, Resistors_THT:R_Array_SIP5, F.Cu at (27.4, 73.7)
- added S1: SPDT, Switches_THT:SW-SPDT-0900766b81587629, F.Cu at (197.6, 22.4)
- added SW1: RESET, Buttons_Switches_ThroughHole:SW_PUSH_6mm_h4.3mm, F.Cu at (172.2, 140.7)
- added SW2: PANIC, Buttons_Switches_ThroughHole:SW_PUSH_6mm_h4.3mm, F.Cu at (185.5, 136.7)
- added U1: WD65C816S_PLCC44, saturn:PLCC-44_THT-Socket, F.Cu at (21.3, 41.1)
- added U10: TL7705B, Housings_DIP:DIP-8_W7.62mm_Socket, F.Cu at (175.3, 121.9)
- added U11: ispMACH4A, saturn:PLCC-44_THT-Socket, F.Cu at (54.9, 36.1)
- added U12: DS1511Y+, Housings_DIP:DIP-28_W15.24mm_Socket, F.Cu at (42.2, 115.3)
- added U13: AS7C34096A, saturn:SOJ-36, F.Cu at (133.6, 71.6)
- added U14: AS7C34096A, saturn:SOJ-36, F.Cu at (106.7, 71.6)
- added U2: AS7C34096A, saturn:SOJ-36, F.Cu at (52.8, 71.6)
- added U3: MAX238, Housings_DIP:DIP-24_W7.62mm_Socket, F.Cu at (148.3, 46.7)
- added U4: SC28L92PLCC44, saturn:PLCC-44_THT-Socket, F.Cu at (136.1, 36.6)
- added U5: AS6C62256A, Housings_DIP:DIP-28_W15.24mm_Socket, F.Cu at (17.3, 103.1)
- added U6: AS7C34096A, saturn:SOJ-36, F.Cu at (79.8, 71.6)
- added U7: WD65C22PLCC44, saturn:PLCC-44_THT-Socket, F.Cu at (109.7, 36.6)
- added U8: WD65C22PLCC44, saturn:PLCC-44_THT-Socket, F.Cu at (81.3, 36.1)
- added U9: 74HC74, Housings_DIP:DIP-14_W7.62mm_Socket, F.Cu at (161.0, 135.1)
- added X1: 3.6864 MHz, Oscillators:Oscillator_DIP-8, F.Cu at (137.7, 122.4)
- added X2: 16MHz, Oscillators:Oscillator_DIP-8, F.Cu at (151.9, 130.0)
Routing:
- added copper zone on GND.Cu, net GND
- added copper zone on VCC.Cu, net VCC
Other:
- board outline added: 206.8 x 138.2 mm

Commit message: Added new footprints. Added docs
Parts:
- removed C23, C24, C25, C26: 0.1uF, Capacitors_ThroughHole:C_Disc_D4.7mm_W2.5mm_P5.00mm
- removed JP1: Enable ISP, Pin_Headers:Pin_Header_Straight_1x02_Pitch2.54mm
- removed U13, U14: AS7C34096A, saturn:SOJ-36
- J1, J2: footprint Connectors_IDC:IDC-Header_2x05_Pitch2.54mm_Angled -> Connectors_IDC:IDC-Header_2x05_Pitch2.54mm_Straight
- J3: footprint Connectors_IDC:IDC-Header_2x07_Pitch2.54mm_Angled -> Connectors_IDC:IDC-Header_2x07_Pitch2.54mm_Straight
- J4, J7: footprint Connectors_IDC:IDC-Header_2x20_Pitch2.54mm_Angled -> Connectors_IDC:IDC-Header_2x20_Pitch2.54mm_Straight
- moved C7 225.2 mm to (246.4, 90.9)
- moved C8 221.1 mm to (239.3, 78.7)
- moved RN2 211.0 mm to (235.7, 107.2)
- moved U5 207.2 mm to (220.0, 59.9), turned to 270 degrees
- moved F2 201.2 mm to (20.3, 30.5), turned to 270 degrees
- moved U1 192.3 mm to (198.1, 116.8)
- moved S1 182.3 mm to (19.3, 60.5), turned to 90 degrees
- moved J5 180.3 mm to (24.4, 26.4)
- moved F1 168.7 mm to (31.0, 30.5), turned to 270 degrees
- moved C19 165.8 mm to (19.3, 67.6), turned to 270 degrees
- moved C15 163.6 mm to (29.0, 132.6)
- moved D1 159.6 mm to (28.4, 57.4), turned to 270 degrees
- moved C9 156.0 mm to (177.3, 67.1)
- moved R4 153.6 mm to (27.4, 63.5)
- moved U12 147.1 mm to (188.0, 96.0), turned to 90 degrees
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Connections:
- RN2 pad 1: Net-(JP1-Pad2) -> VCC
- U11 pad 21: /Glue and control logic/~RAM2 -> Net-(U11-Pad21)
- U11 pad 30: /Glue and control logic/~RAM3 -> Net-(U11-Pad30)
Other:
- board text added: "Expansion port"
- board text added: "IDE"
- board text added: "JTAG"
- board text added: "UART1"
- board text added: "UART2"
- board text added: "VIA"

Commit message: Cosmetic changes to schema. Parking this project as router can't find a route.
Parts:
- moved D4 232.8 mm to (45.2, 162.1), turned to 0 degrees
- moved J6 219.8 mm to (248.4, 100.6), turned to 0 degrees
- moved R7 219.3 mm to (47.2, 155.4), turned to 270 degrees
- moved R6 208.2 mm to (53.8, 156.0), turned to 180 degrees
- moved J7 203.5 mm to (236.7, 131.1), turned to 0 degrees
- moved D1 203.4 mm to (223.0, 116.7), turned to 0 degrees
- moved C19 195.3 mm to (208.9, 114.2), turned to 0 degrees
- moved R4 189.0 mm to (205.3, 127.5)
- moved H2 188.2 mm to (209.7, 121.8)
- moved H4 180.3 mm to (38.6, 162.6)
- moved J5 171.3 mm to (192.0, 61.5), turned to 270 degrees
- moved C17 165.4 mm to (52.8, 124.0), turned to 0 degrees
- moved U5 164.2 mm to (93.0, 164.1), turned to 180 degrees
- moved C15 160.5 mm to (189.4, 129.0), turned to 0 degrees
- moved C22 156.7 mm to (208.9, 108.0), turned to 0 degrees
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Connections:
- J1 pad 1: Net-(J1-Pad1) -> (no net)
- J1 pad 10: Net-(J1-Pad10) -> (no net)
- J1 pad 4: Net-(J1-Pad4) -> (no net)
- J1 pad 6: Net-(J1-Pad6) -> (no net)
- J1 pad 9: Net-(J1-Pad9) -> (no net)
- J2 pad 1: Net-(J2-Pad1) -> (no net)
- J2 pad 10: Net-(J2-Pad10) -> (no net)
- J2 pad 4: Net-(J2-Pad4) -> (no net)
- J2 pad 6: Net-(J2-Pad6) -> (no net)
- J2 pad 9: Net-(J2-Pad9) -> (no net)
- J4 pad 20: Net-(J4-Pad20) -> (no net)
- J4 pad 21: Net-(J4-Pad21) -> (no net)
- J4 pad 27: Net-(J4-Pad27) -> (no net)
- J4 pad 28: Net-(J4-Pad28) -> (no net)
- J4 pad 31: Net-(J4-Pad31) -> (no net)
- J4 pad 34: Net-(J4-Pad34) -> (no net)
- J5 pad 4: Net-(J5-Pad4) -> (no net)
- J6 pad 10: Net-(J6-Pad10) -> (no net)
- J6 pad 9: Net-(J6-Pad9) -> (no net)
- J7 pad 19: Net-(J7-Pad19) -> (no net)
- J7 pad 38: Net-(J7-Pad38) -> (no net)
- S1 pad 3: Net-(S1-Pad3) -> (no net)
- U1 pad 12: Net-(U1-Pad12) -> (no net)
- U1 pad 2: Net-(U1-Pad2) -> (no net)
- U1 pad 39: Net-(U1-Pad39) -> (no net)
- U1 pad 42: Net-(U1-Pad42) -> (no net)
- U1 pad 6: Net-(U1-Pad6) -> (no net)
- U11 pad 21: Net-(U11-Pad21) -> (no net)
- U11 pad 30: Net-(U11-Pad30) -> (no net)
- U12 pad 23: Net-(U12-Pad23) -> (no net)
- U2 pad 19: Net-(U2-Pad19) -> (no net)
- U2 pad 36: Net-(U2-Pad36) -> (no net)
- U4 pad 1: Net-(U4-Pad1) -> (no net)
- U4 pad 15: Net-(U4-Pad15) -> (no net)
- U4 pad 16: Net-(U4-Pad16) -> (no net)
- U4 pad 17: Net-(U4-Pad17) -> (no net)
- U4 pad 23: Net-(U4-Pad23) -> (no net)
- U4 pad 29: Net-(U4-Pad29) -> (no net)
- U4 pad 3: Net-(U4-Pad3) -> (no net)
- U4 pad 30: Net-(U4-Pad30) -> (no net)
- U4 pad 31: Net-(U4-Pad31) -> (no net)
- U4 pad 34: Net-(U4-Pad34) -> (no net)
- U4 pad 37: Net-(U4-Pad37) -> (no net)
- U4 pad 40: Net-(U4-Pad40) -> (no net)
- U4 pad 41: Net-(U4-Pad41) -> (no net)
- U4 pad 42: Net-(U4-Pad42) -> (no net)
- U4 pad 43: Net-(U4-Pad43) -> (no net)
- U6 pad 19: Net-(U6-Pad19) -> (no net)
- U6 pad 36: Net-(U6-Pad36) -> (no net)
- U7 pad 11: Net-(U7-Pad11) -> (no net)
- U7 pad 19: Net-(U7-Pad19) -> (no net)
- U7 pad 20: Net-(U7-Pad20) -> (no net)
- U7 pad 22: Net-(U7-Pad22) -> (no net)
- U7 pad 33: Net-(U7-Pad33) -> (no net)
- U7 pad 38: Net-(U7-Pad38) -> (no net)
- U7 pad 43: Net-(U7-Pad43) -> (no net)
- U7 pad 44: Net-(U7-Pad44) -> (no net)
- U8 pad 11: Net-(U8-Pad11) -> (no net)
- U8 pad 22: Net-(U8-Pad22) -> (no net)
- U8 pad 33: Net-(U8-Pad33) -> (no net)
- U8 pad 38: Net-(U8-Pad38) -> (no net)
- U8 pad 43: Net-(U8-Pad43) -> (no net)
- U8 pad 44: Net-(U8-Pad44) -> (no net)
- U9 pad 8: Net-(U9-Pad8) -> (no net)
- U9 pad 9: Net-(U9-Pad9) -> (no net)
- X1 pad 1: Net-(X1-Pad1) -> (no net)
- X2 pad 1: Net-(X2-Pad1) -> (no net)
Routing:
- removed copper zone on GND.Cu, net GND
- removed copper zone on VCC.Cu, net VCC
Other:
- board outline removed
- board text removed: "Expansion port"
- board text removed: "IDE"
- board text removed: "JTAG"
- board text removed: "UART1"
- board text removed: "UART2"
- board text removed: "VIA"
